File: mcu.kicad_sch (KiCad schematic)
At the start: 40 parts, among them IC1 SN74AHCT1G125DBVR, J201 Connector, USB-TYPE-C-16P, SW201 SK-12D02, U1 STM32F723VET6, U2 USBLC6-2SC6, U201 TS3USB221ARSER, U202 EC11E15244B2, X1 16MHz

Commit message: clean schematics
Parts:
- added J201: SWD_3.3V, Connector_Wire:SolderWirePad_1x01_SMD_2x4mm, symbol Connector:Conn_01x01_Pin
- added J202: SWD_GND, Connector_Wire:SolderWirePad_1x01_SMD_2x4mm, symbol Connector:Conn_01x01_Pin
- added J203: SWD_SWDIO, Connector_Wire:SolderWirePad_1x01_SMD_2x4mm, symbol Connector:Conn_01x01_Pin
- added J204: SWD_SWCLK, Connector_Wire:SolderWirePad_1x01_SMD_2x4mm, symbol Connector:Conn_01x01_Pin
- renumbered J201 to J1, U202 to RV1, SW201 to SW_BOOT, SW_RST1 to SW_RESET, U201 to U3, IC1 to U6
Connections:
- net +3.3V: now also J201.1 (Pin_1)
- net ENCODER_WAVE_1: now also U1.90 (PB4); no longer U1.92 (PB6)
- net ENCODER_WAVE_2: now also U1.91 (PB5); no longer U1.93 (PB7)
- net GND: now also J202.1 (Pin_1)
- net SWDIO: now reaches U1.72 (PA13)
- net SWDIO: now also J203.1 (Pin_1)
- net SWCLK: now reaches U1.76 (PA14)
- net SWCLK: now also J204.1 (Pin_1)
- net ENCODER_SW: now reaches U1.89 (PB3)
- net ENCODER_SW: now also R287.2, RV1.E1 (NO)
- removed net ENCODER_PUSH_BUTTON: R287.2, RV1.E1 (NO), U1.95 (PB8)
- no-connect marks 58 -> 56
Other:
- note added: "LED LEVEL DATA SHIFTER"
- note added: "RESET SWITCH"
- note added: "SOLDER PAD"
- note added: "TODO: - Check differential pairs - Check MCU pinout - Check MCU power supply - Check LDO circuit"
- note added: "USB"
- note added: "USB MULTIPLEXER"
- note removed: "J'ai add ce condo d'après la DS ->"
- note removed: "RESET"
- note removed: "TODO: - Verifier le pinout analogique - Verifier que les 2 ADC peuvent fonctionner en simultanné en DMA avec les bonnes frequences - Verifier les pairs diff USB - Besoin de pin pour les led (timer)"
- note removed: "TODO: CHECK CLOCK FREQUENCY WITH STMCUBEMX"
- note removed: "TODO: CHECK PIN FEATURES WITH CUBEMX"
- note removed: "TODO: VERIFIEIR PIN ADC"
- moved on the sheet: C165, C166, C167, C168, C169, C170, C171, C172, C173, C174, C175, C176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

Commit message: clean PCB
Parts:
- renumbered SW_BOOT to SW_BOOT1, SW_RESET to SW_RESET1
Other:
- note added: "TODO: - Check differential pairs - Check MCU pinout - Check MCU power supply - Check LDO circuit - Emplacement des VIS - Stabilisateur"
- note removed: "TODO: - Check differential pairs - Check MCU pinout - Check MCU power supply - Check LDO circuit"
Changed lines of the file:
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@@
 		)
 	)
-	(text "TODO:\n\n- Check differential pairs\n- Check MCU pinout\n- Check MCU power supply\n- Check LDO circuit"
+	(text "TODO:\n\n- Check differential pairs\n- Check MCU pinout\n- Check MCU power supply\n- Check LDO circuit\n\n- Emplacement des VIS\n- Stabilisateur"
 		(exclude_from_sim no)
 		(at 356.87 33.528 0)
@@
 		(dnp no)
 		(fields_autoplaced yes)
-		(property "Reference" "SW_BOOT"
+		(property "Reference" "SW_BOOT1"
 			(at 31.75 83.1849 90)
 			(effects
@@
 			(project "75he"
 				(path "/0edb4e17-93a4-4f7b-ad91-3a5c72b69d23/e7ec310e-33d9-421e-aaaf-42ca5ffe1b35"
-					(reference "SW_BOOT")
+					(reference "SW_BOOT1")
 					(unit 1)
 				)
@@
 		(dnp no)
 		(fields_autoplaced yes)
-		(property "Reference" "SW_RESET"
+		(property "Reference" "SW_RESET1"
 			(at 95.25 58.42 0)
 			(effects
@@
 			(project "75he"
 				(path "/0edb4e17-93a4-4f7b-ad91-3a5c72b69d23/e7ec310e-33d9-421e-aaaf-42ca5ffe1b35"
-					(reference "SW_RESET")
+					(reference "SW_RESET1")
 					(unit 1)
 				)
