File: screws.kicad_sch (KiCad schematic)
At the start: 12 parts

Commit message: mounting hole
Parts:
- added H13, H14, H15, H16, H17, H18: MountingHole_Pad, MountingHole:MountingHole_2.2mm_M2_ISO14580_Pad, symbol Mechanical:MountingHole_Pad
Connections:
- net GND: now also H13.1, H14.1, H15.1, H16.1, H17.1, H18.1

Commit message: Placed led
Parts:
- renumbered H14 to H10, H9 to H11, H15 to H12, H10 to H13, H16 to H14, H11 to H15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
