File: power_supply.kicad_sch (KiCad schematic)
At the start: 9 parts, among them U4 TPS7A4701RGWR, U5 LDL1117S33R

Commit message: mcu capacitor, usb port, ldo
Parts:
- U5: footprint LDL1117S33R:SOT223_STM -> SOT223_STM
Changed lines of the file:
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@@
 			)
 		)
-		(property "Footprint" "LDL1117S33R:SOT223_STM"
+		(property "Footprint" "SOT223_STM"
 			(at 189.23 124.46 0)
 			(effects

Commit message: Placed led
Parts:
- renumbered C184 to C197, C183 to C198, C187 to C199, C186 to C200, C182 to C201, D267 to LED2, R289 to R91, U4 to U5, U5 to U6

Commit message: led capacitor & sensor capacitor & fixes
Parts:
- U6: footprint SOT223_STM -> LDL1117S33R:SOT223_STM
Changed lines of the file:
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@@
 			)
 		)
-		(property "Footprint" "SOT223_STM"
+		(property "Footprint" "LDL1117S33R:SOT223_STM"
 			(at 189.23 124.46 0)
 			(hide yes)

Commit message: lcsc part
Parts:
- U6: LCSC (none) -> C435835
Changed lines of the file:
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@@
+			)
+		)
+		(property "LCSC" "C435835"
+			(at 189.23 124.46 0)
+			(hide yes)
+			(show_name no)
+			(do_not_autoplace no)
+			(effects
+				(font
+					(size 1.27 1.27)
+				)
 			)
 		)
