File: led.kicad_sch (KiCad schematic)
At the start: 132 parts

Commit message: fixes & doc
Parts:
- added R1: 330Ω, PCM_JLCPCB:R_0603, symbol PCM_JLCPCB-Resistors:0603,330Ω
Connections:
- net LED_DATA_5V: now also R1.1; no longer D201.4 (DIN)
- new net: D201.4 (DIN), R1.2
Other:
- moved on the sheet: C218, C219, C220, C221, C222, C223, C224, C225, C226, C227, C228, C229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

Commit message: Add WS2812 footprints, resistors and net names
Replace generic switch footprints with proper SMD components and metadata: add WS2812B RGB LED footprints (with pads, nets, 3D models and part/Datasheet/LCSC info), add many resistor footprints and detailed properties, and update net names for LED data lines (e.g. Net-(D201-DIN/DOUT) etc.). Also adjust footprint positions, pad assignments, sheet references (LED/HE Sensors), and footprint drawing/printer layers to match correct component geometry for assembly and BOM generation.
Parts:
- renumbered R1 to R290
Changed lines of the file:
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@@
 		(dnp no)
 		(fields_autoplaced yes)
-		(property "Reference" "R?"
+		(property "Reference" "R290"
 			(at 34.29 39.37 90)
 			(effects
@@
 			(project "75he"
 				(path "/0edb4e17-93a4-4f7b-ad91-3a5c72b69d23/84df50b8-8ca3-419c-821a-323741d71109"
-					(reference "R?")
+					(reference "R290")
 					(unit 1)
 				)

Commit message: Placed led
Parts:
- removed D265, D266: WS2812B, PCM_JLCPCB:LED_WS2812B_PLCC4_5.0x5.0mm_P3.2mm, symbol PCM_JLCPCB-Extended:LED, WS2812B, 5050
- added C266, C267, C268, C269, C270, C271, C272, C273, C274, C275, C276, C277, C278, C279, C280, C281: 100nF, PCM_JLCPCB:C_0402, symbol PCM_JLCPCB-Capacitors:0402,100nF
- added D65, D66, D67, D68, D69, D70, D71, D72, D73, D74, D75, D76, D77, D78, D79, D80, D81, D82: WS2812B, PCM_JLCPCB:LED_WS2812B_PLCC4_5.0x5.0mm_P3.2mm, symbol PCM_JLCPCB-Extended:LED, WS2812B, 5050
- renumbered C218 to C202, C219 to C203, C220 to C204, C221 to C205, C222 to C206, C223 to C207, C224 to C208, C225 to C209, C226 to C210, C227 to C211, C228 to C212, C229 to C213, C230 to C214, C231 to C215, C232 to C216, C233 to C217, C234 to C218, C235 to C219, C236 to C220, C237 to C221, C238 to C222, C239 to C223, C240 to C224, C241 to C225, C242 to C226, C243 to C227, C244 to C228, C245 to C229, C246 to C230, C247 to C231, C248 to C232, C249 to C233, C250 to C234, C254 to C235, C258 to C236, C262 to C237, C266 to C238, C270 to C239, C274 to C240, C278 to C241, C251 to C242, C255 to C243, C259 to C244, C263 to C245, C267 to C246, C271 to C247, C275 to C248, C279 to C249, C252 to C250, C256 to C251, C260 to C252, C264 to C253, C268 to C254, C272 to C255, C276 to C256, C280 to C257, C253 to C258, C257 to C259, C261 to C260, C265 to C261, C269 to C262, C273 to C263, C277 to C264, C281 to C265, D201 to D1, D210 to D10, D211 to D11, D212 to D12, D213 to D13, D214 to D14, D215 to D15, D216 to D16, D217 to D17, D218 to D18, D219 to D19, D202 to D2, D220 to D20, D221 to D21, D222 to D22, D223 to D23, D224 to D24, D225 to D25, D226 to D26, D227 to D27, D228 to D28, D229 to D29, D203 to D3, D230 to D30, D231 to D31, D232 to D32, D233 to D33, D237 to D34, D241 to D35, D245 to D36, D249 to D37, D253 to D38, D257 to D39, D204 to D4, D261 to D40, D234 to D41, D238 to D42, D242 to D43, D246 to D44, D250 to D45, D254 to D46, D258 to D47, D262 to D48, D235 to D49, D205 to D5, D239 to D50, D243 to D51, D247 to D52, D251 to D53, D255 to D54, D259 to D55, D263 to D56, D236 to D57, D240 to D58, D244 to D59, D206 to D6, D248 to D60, D252 to D61, D256 to D62, D260 to D63, D264 to D64, D207 to D7, D208 to D8, D209 to D9, R290 to R92
Connections:
- net +5V: now also C266.1, C267.1, C268.1, C269.1, C270.1, C271.1, C272.1, C273.1, C274.1, C275.1, C276.1, C277.1, C278.1, C279.1, C280.1, C281.1, D65.1 (VDD), D66.1 (VDD), D67.1 (VDD), D68.1 (VDD), D69.1 (VDD), D70.1 (VDD), D71.1 (VDD), D72.1 (VDD), D73.1 (VDD), D74.1 (VDD), D75.1 (VDD), D76.1 (VDD), D77.1 (VDD), D78.1 (VDD), D79.1 (VDD), D80.1 (VDD), D81.1 (VDD), D82.1 (VDD)
- net GND: now also C266.2, C267.2, C268.2, C269.2, C270.2, C271.2, C272.2, C273.2, C274.2, C275.2, C276.2, C277.2, C278.2, C279.2, C280.2, C281.2, D65.3 (VSS), D66.3 (VSS), D67.3 (VSS), D68.3 (VSS), D69.3 (VSS), D70.3 (VSS), D71.3 (VSS), D72.3 (VSS), D73.3 (VSS), D74.3 (VSS), D75.3 (VSS), D76.3 (VSS), D77.3 (VSS), D78.3 (VSS), D79.3 (VSS), D80.3 (VSS), D81.3 (VSS), D82.3 (VSS)
- net at D64.2 (DOUT): now also D65.4 (DIN)
- new net: D81.2 (DOUT), D82.4 (DIN)
- new net: D80.2 (DOUT), D81.4 (DIN)
- new net: D68.2 (DOUT), D69.4 (DIN)
- new net: D67.2 (DOUT), D68.4 (DIN)
- new net: D69.2 (DOUT), D70.4 (DIN)
- new net: D70.2 (DOUT), D71.4 (DIN)
- new net: D76.2 (DOUT), D77.4 (DIN)
- new net: D75.2 (DOUT), D76.4 (DIN)
- new net: D66.2 (DOUT), D67.4 (DIN)
- new net: D65.2 (DOUT), D66.4 (DIN)
- new net: D77.2 (DOUT), D78.4 (DIN)
- new net: D74.2 (DOUT), D75.4 (DIN)
- new net: D73.2 (DOUT), D74.4 (DIN)
- new net: D78.2 (DOUT), D79.4 (DIN)
- new net: D72.2 (DOUT), D73.4 (DIN)
- new net: D71.2 (DOUT), D72.4 (DIN)
- new net: D79.2 (DOUT), D80.4 (DIN)

Commit message: route sensors to mux & data led
Connections:
- net at D29.2 (DOUT): now also D28.4 (DIN); no longer D30.4 (DIN)
- net at D28.2 (DOUT): now also D27.4 (DIN); no longer D29.4 (DIN)
- net at D81.2 (DOUT): now also D80.4 (DIN); no longer D82.4 (DIN)
- net at D81.4 (DIN): now also D82.2 (DOUT); no longer D80.2 (DOUT)
- net at D45.4 (DIN): now also D46.2 (DOUT); no longer D44.2 (DOUT)
- net at D47.2 (DOUT): now also D46.4 (DIN); no longer D48.4 (DIN)
- net at D47.4 (DIN): now also D48.2 (DOUT); no longer D46.2 (DOUT)
- net at D25.2 (DOUT): now also D24.4 (DIN); no longer D26.4 (DIN)
- net at D25.4 (DIN): now also D26.2 (DOUT); no longer D24.2 (DOUT)
- net at D27.2 (DOUT): now also D26.4 (DIN); no longer D28.4 (DIN)
- net at D16.4 (DIN): now also D17.2 (DOUT); no longer D15.2 (DOUT)
- net at D15.4 (DIN): now also D16.2 (DOUT); no longer D14.2 (DOUT)
- net at D20.2 (DOUT): now also D19.4 (DIN); no longer D21.4 (DIN)
- net at D20.4 (DIN): now also D21.2 (DOUT); no longer D19.2 (DOUT)
- net at D22.2 (DOUT): now also D21.4 (DIN); no longer D23.4 (DIN)
- net at D22.4 (DIN): now also D23.2 (DOUT); no longer D21.2 (DOUT)
- net at D18.2 (DOUT): now also D17.4 (DIN); no longer D19.4 (DIN)
- net at D18.4 (DIN): now also D19.2 (DOUT); no longer D17.2 (DOUT)
- net at D76.2 (DOUT): now also D75.4 (DIN); no longer D77.4 (DIN)
- net at D76.4 (DIN): now also D77.2 (DOUT); no longer D75.2 (DOUT)
- net at D55.2 (DOUT): now also D54.4 (DIN); no longer D56.4 (DIN)
- net at D55.4 (DIN): now also D56.2 (DOUT); no longer D54.2 (DOUT)
- net at D57.4 (DIN): now also D58.2 (DOUT); no longer D56.2 (DOUT)
- net at D78.4 (DIN): now also D79.2 (DOUT); no longer D77.2 (DOUT)
- net at D52.2 (DOUT): now also D51.4 (DIN); no longer D53.4 (DIN)
- net at D52.4 (DIN): now also D53.2 (DOUT); no longer D51.2 (DOUT)
- net at D49.2 (DOUT): now also D48.4 (DIN); no longer D50.4 (DIN)
- net at D49.4 (DIN): now also D50.2 (DOUT); no longer D48.2 (DOUT)
- net LED_DATA_OUT_4: now reaches D45.2 (DOUT)
- net LED_DATA_OUT_4: now also D59.4 (DIN), D72.2 (DOUT), D82.4 (DIN); no longer D46.4 (DIN)
- net at D57.2 (DOUT): now also D56.4 (DIN); no longer D58.4 (DIN)
- net at D74.2 (DOUT): now also D73.4 (DIN); no longer D75.4 (DIN)
- net at D74.4 (DIN): now also D75.2 (DOUT); no longer D73.2 (DOUT)
- net at D78.2 (DOUT): now also D77.4 (DIN); no longer D79.4 (DIN)
- new net: D23.4 (DIN), D24.2 (DOUT)
- new net: D53.4 (DIN), D54.2 (DOUT)
- new net: D50.4 (DIN), D51.2 (DOUT)
- new net: D79.4 (DIN), D80.2 (DOUT)
- new net LED_DATA_OUT_1: D14.2 (DOUT), D29.4 (DIN)
- new net LED_DATA_OUT_2: D15.2 (DOUT), D30.4 (DIN)
- new net LED_DATA_OUT_3: D44.2 (DOUT), D58.4 (DIN)
Other:
- moved on the sheet: C216, C217, C218, C219, C220, C221, C222, C223, C224, C225, C226, C227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

Commit message: cleanup
Connections:
- net LED_DATA_OUT_4: no longer D72.2 (DOUT), D82.4 (DIN)
- new net LED_DATA_OUT_5: D72.2 (DOUT), D82.4 (DIN)
Other:
- moved on the sheet: C210, C211, C212, C213, C214, C215, C216, C217, C218, C219, C220, C221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
