File: legacy/proto-mcu-v1/mcu.kicad_sch (KiCad schematic)
At the start: 81 parts, among them IC1 SN74AHCT1G125DBVR, J1 Connector, USB-TYPE-C-16P, J2 TSW-104-07-F-S, SW1 SSSF111800, U2 AMS1117, U3 USBLC6-2SC6, U4 STM32F723ZET6, X1 16Mhz

Commit message: Reorganize KiCad libraries; add Legacy Docs
Large repository reorganization of KiCad assets: added Docs and Legacy/ proto directories with many component datasheets and legacy project files, moved and renamed numerous footprints, 3D models and symbol files into consolidated Library/ and Legacy/ paths, and removed outdated/duplicate files. Purpose is to centralize libraries, preserve legacy designs, and clean up footprint/3D model locations for easier maintenance.
Parts:
- IC1: footprint SamacSys_Parts:SOT95P280X145-5N -> SN74AHCT1G125DBVR:SOT95P280X145-5N; symbol SamacSys_Parts:SN74AHCT1G125DBVR -> SN74AHCT1G125DBVR:SN74AHCT1G125DBVR
- SW1: footprint easyeda2kicad:SW-TH_SSSF111800 -> SSSF111800:SW-TH_SSSF111800; symbol easyeda2kicad:SSSF111800 -> SSSF111800:SSSF111800
Changed lines of the file:
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@@
 	)
 	(symbol
-		(lib_id "SamacSys_Parts:SN74AHCT1G125DBVR")
+		(lib_id "SN74AHCT1G125DBVR:SN74AHCT1G125DBVR")
 		(at 129.54 196.85 180)
 		(unit 1)
@@
 			)
 		)
-		(property "Footprint" "SamacSys_Parts:SOT95P280X145-5N"
+		(property "Footprint" "SN74AHCT1G125DBVR:SOT95P280X145-5N"
 			(at 107.95 101.93 0)
 			(effects
@@
 	)
 	(symbol
-		(lib_id "easyeda2kicad:SSSF111800")
+		(lib_id "SSSF111800:SSSF111800")
 		(at 99.06 73.66 90)
 		(unit 1)
@@
 			)
 		)
-		(property "Footprint" "easyeda2kicad:SW-TH_SSSF111800"
+		(property "Footprint" "SSSF111800:SW-TH_SSSF111800"
 			(at 111.76 73.66 0)
 			(effects
