File: legacy/proto-mcu-v2/mcu.kicad_pcb (KiCad board)
At the start: 2 copper layers, 55 x 41 mm, 74 parts, among them IC1 SN74AHCT1G125DBVR, J1 Connector, USB-TYPE-C-16P, J2 TSW-104-07-F-S, SW2 SK-12D02, U1 STM32F723VET6, U2 AMS1117, U3 USBLC6-2SC6, U5 TS3USB221ARSER, X1 16Mhz

Commit message: Reorganize KiCad libraries; add Legacy Docs
Large repository reorganization of KiCad assets: added Docs and Legacy/ proto directories with many component datasheets and legacy project files, moved and renamed numerous footprints, 3D models and symbol files into consolidated Library/ and Legacy/ paths, and removed outdated/duplicate files. Purpose is to centralize libraries, preserve legacy designs, and clean up footprint/3D model locations for easier maintenance.
Parts:
- IC1: footprint SamacSys_Parts:SOT95P280X145-5N -> SN74AHCT1G125DBVR:SOT95P280X145-5N
- SW2: footprint easyeda2kicad:SW-TH_SK-12D02VG3 -> SW-TH_SK-12D02VG3:SW-TH_SK-12D02VG3
- U5: footprint footprints:RSE10 -> TS3USB221ARSER:RSE10
Changed lines of the file:
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@@
 		)
 		(embedded_fonts no)
-		(model "${KIPRJMOD}/../../Library/3D/JLCPCB.3dshapes/C_0805.step"
+		(model "${KIPRJMOD}/Library/3D/JLCPCB.3dshapes/C_0805.step"
 			(offset
 				(xyz 0 0 0)
@@
 		)
 		(embedded_fonts no)
-		(model "${KIPRJMOD}/../../Library/3D/JLCPCB.3dshapes/R_0402.step"
+		(model "${KIPRJMOD}/Library/3D/JLCPCB.3dshapes/R_0402.step"
 			(offset
 				(xyz 0 0 0)
@@
 		)
 		(embedded_fonts no)
-		(model "${KIPRJMOD}/../../Library/1812L300_24SLER/3D/1812L300_24SLER.stp"
+		(model "${KIPRJMOD}/Library/3D/1812L300_24SLER/1812L300_24SLER.stp"
 			(offset
 				(xyz 0 0 0)
@@
 		)
 		(embedded_fonts no)
-		(model "${KIPRJMOD}/../../Library/3D/JLCPCB.3dshapes/D_0603.step"
+		(model "${KIPRJMOD}/Library/3D/JLCPCB.3dshapes/D_0603.step"
 			(offset
 				(xyz 0 0 0)
@@
 		)
 		(embedded_fonts no)
-		(model "${KIPRJMOD}/../../Library/3D/JLCPCB.3dshapes/C_0603.step"
+		(model "${KIPRJMOD}/Library/3D/JLCPCB.3dshapes/C_0603.step"
 			(offset
 				(xyz 0 0 0)
@@
 		)
 		(embedded_fonts no)
-		(model "${KIPRJMOD}/../../Library/3D/KiCad/Package_QFP.3dshapes/LQFP-100_14x14mm_P0.5mm.step"
+		(model "${KIPRJMOD}/Library/3D/KiCad/Package_QFP.3dshapes/LQFP-100_14x14mm_P0.5mm.step"
 			(offset
 				(xyz 0 0 0)
@@
 		)
 		(embedded_fonts no)
-		(model "${KIPRJMOD}/../../Library/3D/JLCPCB.3dshapes/C_0805.step"
+		(model "${KIPRJMOD}/Library/3D/JLCPCB.3dshapes/C_0805.step"
 			(offset
 				(xyz 0 0 0)
@@
 		)
 		(embedded_fonts no)
-		(model "${KIPRJMOD}/../../Library/3D/JLCPCB.3dshapes/C_0603.step"
+		(model "${KIPRJMOD}/Library/3D/JLCPCB.3dshapes/C_0603.step"
 			(offset
 				(xyz 0 0 0)
@@
 		)
 		(embedded_fonts no)
-		(model "${KIPRJMOD}/../../Library/3D/JLCPCB.3dshapes/R_0402.step"
+		(model "${KIPRJMOD}/Library/3D/JLCPCB.3dshapes/R_0402.step"
 			(offset
 				(xyz 0 0 0)
@@
 		)
 		(embedded_fonts no)
-		(model "${KIPRJMOD}/../../Library/LDL1117S33R/3D/LDL1117S33R.stp"
+		(model "${KIPRJMOD}/Library/3D/LDL1117S33R/LDL1117S33R.stp"
 			(offset
 				(xyz 0 -3.25 0)
@@
 		)
 		(embedded_fonts no)
-		(model "${KIPRJMOD}/../../Library/3D/JLCPCB.3dshapes/C_0805.step"
+		(model "${KIPRJMOD}/Library/3D/JLCPCB.3dshapes/C_0805.step"
 			(offset
 				(xyz 0 0 0)
@@
 		)
 		(embedded_fonts no)
-		(model "${KIPRJMOD}/../../Library/3D/JLCPCB.3dshapes/D_0805.step"
+		(model "${KIPRJMOD}/Library/3D/JLCPCB.3dshapes/D_0805.step"
 			(offset
 				(xyz 0 0 0)
@@
 		)
 		(embedded_fonts no)
-		(model "${KIPRJMOD}/../../Library/3D/JLCPCB.3dshapes/C_0805.step"
+		(model "${KIPRJMOD}/Library/3D/JLCPCB.3dshapes/C_0805.step"
 			(offset
 				(xyz 0 0 0)
@@
 		(embedded_fonts no)
 	)
-	(footprint "SamacSys_Parts:SOT95P280X145-5N"
+	(footprint "SN74AHCT1G125DBVR:SOT95P280X145-5N"
 		(layer "F.Cu")
 		(at 166.41 112.68)
@@
 		)
 		(embedded_fonts no)
-		(model "C:\\Users\\ferre\\Codespace\\Projects\\hall-effect-keyboard\\mcu\\SamacSys_Parts.3dshapes\\SN74AHCT1G125DBVR.stp"
+		(model "${KIPRJMOD}/Library/3D/SN74AHCT1G125DBVR/SN74AHCT1G125DBVR.stp"
 			(offset
 				(xyz 0 0 0)
@@
 		)
 		(embedded_fonts no)
-		(model "${KIPRJMOD}/../../Library/3D/JLCPCB.3dshapes/TYPE-C-SMD_HX-TYPE-C-16PIN.step"
+		(model "${KIPRJMOD}/Library/3D/JLCPCB.3dshapes/TYPE-C-SMD_HX-TYPE-C-16PIN.step"
 			(offset
 				(xyz 0 -1.063 0)
@@
 		)
 		(embedded_fonts no)
-		(model "${KIPRJMOD}/../../Library/3D/JLCPCB.3dshapes/C_0603.step"
+		(model "${KIPRJMOD}/Library/3D/JLCPCB.3dshapes/C_0603.step"
 			(offset
 				(xyz 0 0 0)
@@
 		)
 		(embedded_fonts no)
-		(model "${KIPRJMOD}/../../Library/3D/KiCad/Package_TO_SOT_SMD.3dshapes/SOT-23-6.step"
+		(model "${KIPRJMOD}/Library/3D/KiCad/Package_TO_SOT_SMD.3dshapes/SOT-23-6.step"
 			(offset
 				(xyz 0 0 0)
@@
 		)
 		(embedded_fonts no)
-		(model "${KIPRJMOD}/../../Library/3D/JLCPCB.3dshapes/C_0805.step"
+		(model "${KIPRJMOD}/Library/3D/JLCPCB.3dshapes/C_0805.step"
 			(offset
 				(xyz 0 0 0)
@@
 		)
 		(embedded_fonts no)
-		(model "${KIPRJMOD}/../../Library/3D/JLCPCB.3dshapes/C_0603.step"
+		(model "${KIPRJMOD}/Library/3D/JLCPCB.3dshapes/C_0603.step"
 			(offset
 				(xyz 0 0 0)
@@
 		)
 		(embedded_fonts no)
-		(model "${KIPRJMOD}/../../Library/3D/KiCad/Connector_PinHeader_2.54mm.3dshapes/PinHeader_1x04_P2.54mm_Vertical.step"
+		(model "${KIPRJMOD}/Library/3D/KiCad/Connector_PinHeader_2.54mm.3dshapes/PinHeader_1x04_P2.54mm_Vertical.step"
 			(offset
 				(xyz 0 0 0)
@@
 		)
 		(embedded_fonts no)
-		(model "${KIPRJMOD}/../../Library/3D/JLCPCB.3dshapes/R_0402.step"
+		(model "${KIPRJMOD}/Library/3D/JLCPCB.3dshapes/R_0402.step"
 			(offset
 				(xyz 0 0 0)
@@
 		)
 		(embedded_fonts no)
-		(model "${KIPRJMOD}/../../Library/3D/JLCPCB.3dshapes/C_0603.step"
+		(model "${KIPRJMOD}/Library/3D/JLCPCB.3dshapes/C_0603.step"
 			(offset
 				(xyz 0 0 0)
@@
 		)
 		(embedded_fonts no)
-		(model "${KIPRJMOD}/../../Library/3D/JLCPCB.3dshapes/C_0603.step"
+		(model "${KIPRJMOD}/Library/3D/JLCPCB.3dshapes/C_0603.step"
 			(offset
 				(xyz 0 0 0)
@@
 		)
 		(embedded_fonts no)
-		(model "${KIPRJMOD}/../../Library/3D/JLCPCB.3dshapes/C_0805.step"
+		(model "${KIPRJMOD}/Library/3D/JLCPCB.3dshapes/C_0805.step"
 			(offset
 				(xyz 0 0 0)
@@
 		)
 		(embedded_fonts no)
-		(model "${KIPRJMOD}/../../Library/3D/JLCPCB.3dshapes/C_0603.step"
+		(model "${KIPRJMOD}/Library/3D/JLCPCB.3dshapes/C_0603.step"
 			(offset
 				(xyz 0 0 0)
@@
 		)
 		(embedded_fonts no)
-		(model "${KIPRJMOD}/../../Library/3D/JLCPCB.3dshapes/C_0603.step"
+		(model "${KIPRJMOD}/Library/3D/JLCPCB.3dshapes/C_0603.step"
 			(offset
 				(xyz 0 0 0)
@@
 		)
 		(embedded_fonts no)
-		(model "${KIPRJMOD}/../../Library/3D/JLCPCB.3dshapes/C_0603.step"
+		(model "${KIPRJMOD}/Library/3D/JLCPCB.3dshapes/C_0603.step"
 			(offset
 				(xyz 0 0 0)
@@
 		)
 		(embedded_fonts no)
-		(model "${KIPRJMOD}/../../Library/3D/JLCPCB.3dshapes/R_0402.step"
+		(model "${KIPRJMOD}/Library/3D/JLCPCB.3dshapes/R_0402.step"
 			(offset
 				(xyz 0 0 0)
@@
 		)
 		(embedded_fonts no)
-		(model "${KIPRJMOD}/../../Library/3D/JLCPCB.3dshapes/C_0805.step"
+		(model "${KIPRJMOD}/Library/3D/JLCPCB.3dshapes/C_0805.step"
 			(offset
 				(xyz 0 0 0)
@@
 		)
 		(embedded_fonts no)
-		(model "${KIPRJMOD}/../../Library/3D/JLCPCB.3dshapes/C_0603.step"
+		(model "${KIPRJMOD}/Library/3D/JLCPCB.3dshapes/C_0603.step"
 			(offset
 				(xyz 0 0 0)
@@
 		)
 		(embedded_fonts no)
-		(model "${KIPRJMOD}/../../Library/3D/KiCad/Inductor_SMD.3dshapes/L_0603_1608Metric.step"
+		(model "${KIPRJMOD}/Library/3D/KiCad/Inductor_SMD.3dshapes/L_0603_1608Metric.step"
 			(offset
 				(xyz 0 0 0)
@@
 		)
 		(embedded_fonts no)
-		(model "${KIPRJMOD}/../../Library/3D/KiCad/Crystal.3dshapes/Crystal_SMD_2520-4Pin_2.5x2.0mm.step"
+		(model "${KIPRJMOD}/Library/3D/KiCad/Crystal.3dshapes/Crystal_SMD_2520-4Pin_2.5x2.0mm.step"
 			(offset
 				(xyz 0 0 0)
@@
 		)
 		(embedded_fonts no)
-		(model "${KIPRJMOD}/../../Library/3D/JLCPCB.3dshapes/C_0603.step"
+		(model "${KIPRJMOD}/Library/3D/JLCPCB.3dshapes/C_0603.step"
 			(offset
 				(xyz 0 0 0)
@@
 		)
 	)
-	(footprint "easyeda2kicad:SW-TH_SK-12D02VG3"
+	(footprint "SW-TH_SK-12D02VG3:SW-TH_SK-12D02VG3"
 		(layer "F.Cu")
 		(at 177.715 104.58 90)
@@
 		)
 		(embedded_fonts no)
-		(model "${KIPRJMOD}/../../Library/SW-TH_SK-12D02VG3/SW-TH_SK-12D02VG3.step"
+		(model "${KIPRJMOD}/Library/3D/SW-TH_SK-12D02VG3/SW-TH_SK-12D02VG3.step"
 			(offset
 				(xyz 0 0 0)
@@
 		)
 		(embedded_fonts no)
-		(model "${KIPRJMOD}/../../Library/3D/JLCPCB.3dshapes/C_0805.step"
+		(model "${KIPRJMOD}/Library/3D/JLCPCB.3dshapes/C_0805.step"
 			(offset
 				(xyz 0 0 0)
@@
 		)
 		(embedded_fonts no)
-		(model "${KIPRJMOD}/../../Library/3D/KiCad/Resistor_SMD.3dshapes/R_0805_2012Metric.step"
+		(model "${KIPRJMOD}/Library/3D/KiCad/Resistor_SMD.3dshapes/R_0805_2012Metric.step"
 			(offset
 				(xyz 0 0 0)
@@
 		)
 	)
-	(footprint "footprints:RSE10"
+	(footprint "TS3USB221ARSER:RSE10"
 		(layer "F.Cu")
 		(at 166.08 116.81)
@@
 		)
 		(embedded_fonts no)
-		(model "${KIPRJMOD}/../../Library/TS3USB221ARSER/3D/TS3USB221ARSER.stp"
+		(model "${KIPRJMOD}/Library/3D/TS3USB221ARSER/TS3USB221ARSER.stp"
 			(offset
 				(xyz 0 0 0)
@@
 		)
 		(embedded_fonts no)
-		(model "${KIPRJMOD}/../../Library/3D/JLCPCB.3dshapes/C_0805.step"
+		(model "${KIPRJMOD}/Library/3D/JLCPCB.3dshapes/C_0805.step"
 			(offset
 				(xyz 0 0 0)
@@
 		)
 		(embedded_fonts no)
-		(model "${KIPRJMOD}/../../Library/3D/JLCPCB.3dshapes/C_0603.step"
+		(model "${KIPRJMOD}/Library/3D/JLCPCB.3dshapes/C_0603.step"
 			(offset
 				(xyz 0 0 0)
@@
 		)
 		(embedded_fonts no)
-		(model "${KIPRJMOD}/../../Library/3D/JLCPCB.3dshapes/D_0603.step"
+		(model "${KIPRJMOD}/Library/3D/JLCPCB.3dshapes/D_0603.step"
 			(offset
 				(xyz 0 0 0)
@@
 		)
 		(embedded_fonts no)
-		(model "${KIPRJMOD}/../../Library/3D/JLCPCB.3dshapes/TS-1088-AR02016.step"
+		(model "${KIPRJMOD}/Library/3D/JLCPCB.3dshapes/TS-1088-AR02016.step"
 			(offset
 				(xyz 0 0 0)
@@
 		)
 		(embedded_fonts no)
-		(model "${KIPRJMOD}/../../Library/3D/JLCPCB.3dshapes/R_0402.step"
+		(model "${KIPRJMOD}/Library/3D/JLCPCB.3dshapes/R_0402.step"
 			(offset
 				(xyz 0 0 0)
@@
 		)
 		(embedded_fonts no)
-		(model "${KIPRJMOD}/../../Library/3D/JLCPCB.3dshapes/C_0402.step"
+		(model "${KIPRJMOD}/Library/3D/JLCPCB.3dshapes/C_0402.step"
 			(offset
 				(xyz 0 0 0)
@@
 		)
 		(embedded_fonts no)
-		(model "${KIPRJMOD}/../../Library/3D/JLCPCB.3dshapes/R_0402.step"
+		(model "${KIPRJMOD}/Library/3D/JLCPCB.3dshapes/R_0402.step"
 			(offset
 				(xyz 0 0 0)
