File: legacy/proto-mcu-v2/mcu.kicad_sch (KiCad schematic)
At the start: 72 parts, among them IC1 SN74AHCT1G125DBVR, J1 Connector, USB-TYPE-C-16P, J2 TSW-104-07-F-S, SW2 SK-12D02, U1 STM32F723VET6, U2 AMS1117, U3 USBLC6-2SC6, U5 TS3USB221ARSER, X1 16Mhz

Commit message: Reorganize KiCad libraries; add Legacy Docs
Large repository reorganization of KiCad assets: added Docs and Legacy/ proto directories with many component datasheets and legacy project files, moved and renamed numerous footprints, 3D models and symbol files into consolidated Library/ and Legacy/ paths, and removed outdated/duplicate files. Purpose is to centralize libraries, preserve legacy designs, and clean up footprint/3D model locations for easier maintenance.
Parts:
- IC1: footprint SamacSys_Parts:SOT95P280X145-5N -> SN74AHCT1G125DBVR:SOT95P280X145-5N; symbol SamacSys_Parts:SN74AHCT1G125DBVR -> SN74AHCT1G125DBVR:SN74AHCT1G125DBVR
- SW2: footprint easyeda2kicad:SW-TH_SK-12D02VG3 -> SW-TH_SK-12D02VG3:SW-TH_SK-12D02VG3; symbol easyeda2kicad:SK-12D02 -> SW-TH_SK-12D02VG3:SK-12D02
- U5: footprint footprints:RSE10 -> TS3USB221ARSER:RSE10; symbol 2025-12-06_14-23-22:TS3USB221ARSER -> TS3USB221ARSER:TS3USB221ARSER
Changed lines of the file:
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@@
 	)
 	(symbol
-		(lib_id "2025-12-06_14-23-22:TS3USB221ARSER")
+		(lib_id "TS3USB221ARSER:TS3USB221ARSER")
 		(at 234.95 152.4 0)
 		(unit 1)
@@
 			)
 		)
-		(property "Footprint" "footprints:RSE10"
+		(property "Footprint" "TS3USB221ARSER:RSE10"
 			(at 234.95 152.4 0)
 			(effects
@@
 	)
 	(symbol
-		(lib_id "easyeda2kicad:SK-12D02")
+		(lib_id "SW-TH_SK-12D02VG3:SK-12D02")
 		(at 68.58 85.09 270)
 		(unit 1)
@@
 			)
 		)
-		(property "Footprint" "easyeda2kicad:SW-TH_SK-12D02VG3"
+		(property "Footprint" "SW-TH_SK-12D02VG3:SW-TH_SK-12D02VG3"
 			(at 58.42 85.09 0)
 			(effects
@@
 	)
 	(symbol
-		(lib_id "SamacSys_Parts:SN74AHCT1G125DBVR")
+		(lib_id "SN74AHCT1G125DBVR:SN74AHCT1G125DBVR")
 		(at 241.3 180.34 0)
 		(unit 1)
@@
 			)
 		)
-		(property "Footprint" "SamacSys_Parts:SOT95P280X145-5N"
+		(property "Footprint" "SN74AHCT1G125DBVR:SOT95P280X145-5N"
 			(at 262.89 275.26 0)
 			(effects
